File: KiCad/Z80-SBC.sch (KiCad schematic (older format))
At the start: 81 parts, among them P1 POWER, P2 RESET, P3 SERIAL, P4 PARALLEL, P5 FLOPPY, P6 5V, SW1 RESET, U1 Z80-CPU, U10 74LS174, U11 74LS174, U12 74F139, U13 74LS138, U14 74LS125, U15 74LS32, U16 74LS32, U17 74LS32, U18 74LS14, U19 74LS14, U2 29F040, U20 74LS06, U21 4MHz, U22 1.8432MHz, U23 8MHz, U24 MAX232A, U25 DS1302, U26 DS1210, U3 AS6C4008, U4 16550, U5 8255, U6 FDC9266, U7 74LS273, U8 74LS240, U9 74LS174, X1 32768Hz

Commit message: Add V2 website materials, unpack the 2.0 gerber and KiCad directories from zip
Parts:
- removed C20, C21, C22, C23: 0.1uF, symbol C
- removed JP3: FDC INT/NMI, symbol JUMPER3
- removed P3: SERIAL, symbol DB9
- removed U10, U9: 74LS174, symbol 74LS174
- removed U12: 74F139, symbol 74LS139
- removed U15, U17: 74LS32, symbol 74LS32
- removed unit 6 of U18
- removed U19: 74LS14, symbol 74LS14
- removed U20: 74LS06, symbol 74LS06
- removed U21: 4MHz, symbol OSC
- removed U22: 1.8432MHz, symbol OSC
- removed U23: 8MHz, symbol OSC
- removed U6: FDC9266, symbol FDC9266
- removed U7: 74LS273, symbol 74LS273
- removed U8: 74LS240, symbol 74LS240
- added P3: SERIAL, symbol CONN_DE9
- added RR2: 1k, symbol RR5
- added RR3: 4.7k, symbol RR5
- added U11: 74ALS139, symbol 74LS139
- added U14: 74LS74, symbol 74LS74
- added unit 6 of U16
- added U17: 8MHz, symbol OSC_DIP14_DIP8
- added U18: 1.8432, symbol OSC_DIP14_DIP8
- added U19: 16MHz, symbol OSC_DIP14_DIP8
- added U6: WD37C65C, symbol 37C65
- added U7: Z84C30, symbol Z84C30
- added U8, U9: 74LS670, symbol 74LS670
- U1: value Z80-CPU -> Z84C00
- U2: value 29F040 -> ST39SF040
- U20: renamed from U24; value MAX232A -> MAX202
- U4: value 16550 -> PC16550D
- U5: value 8255 -> CP82C55A
- renumbered C24 to C20, C25 to C21, C26 to C22, C27 to C23, C28 to C24, C29 to C25, C30 to C26, RR2 to RR1, RR1 to RR4, U11 to U10, U13 to U12, U14 to U13, U16 to U15, U18 to U16, U25 to U21, U26 to U22
Connections:
- net ROM_A15 is gone; now on net MA15: U2.3 (A15)
- net ROM_A16 is gone; now on net MA16: U2.2 (A16)
- net ROM_A17 is gone; now on net MA17: U2.30 (A17)
- net ROM_A18 is gone; now on net MA18: U2.1 (A18)
- net A0: now also U6.4 (A0), U7.18 (CS0), U8.14 (WA), U9.14 (WA)
- net A1: now also U7.19 (CS1), U8.13 (WB), U9.13 (WB)
- net A14: now also U8.5 (RA), U9.5 (RA); no longer U2.29 (A14), U3.3 (A14)
- net A15: now also U8.4 (RB), U9.4 (RB)
- net A2: now also U11.14 (A)
- net A7: now also U15.10
- net CPU_CLK: now also U17.8 (OUT), U7.15 (CLK)
- net D0: now also U10.6 (D2), U13.8, U14.2 (D), U6.7 (DB0), U7.25 (D0), U8.15 (D1); no longer U13.11, U13.3
- net D1: now also U6.8 (DB1), U7.26 (D1), U8.1 (D2)
- net D2: now also U6.9 (DB2), U7.27 (D2), U8.2 (D3); no longer U10.6 (D2)
- net D3: now also U10.11 (D3), U6.10 (DB3), U7.28 (D3), U8.3 (D4); no longer U10.14 (D5)
- net D4: now also U6.11 (DB4), U7.1 (D4), U9.15 (D1)
- net D5: now also U10.3 (D0), U6.12 (DB5), U7.2 (D5), U9.1 (D2); no longer U10.4 (D1)
- net D6: now also U10.14 (D5), U13.3, U6.13 (DB6), U7.3 (D6), U9.2 (D3); no longer U10.11 (D3), U13.8
- net D7: now also U10.4 (D1), U13.6, U6.14 (DB7), U7.4 (D7), U9.3 (D4); no longer U10.3 (D0)
- net FDC_CLK: now also U19.8 (OUT), U6.23 (CLK1)
- net GND: now also U4.37 (~DSR), P3.5, P3.GND, RR2.1 (COM), RR3.1 (COM), U11.8 (GND), U11.8 (GND), U14.7 (GND), U14.7 (GND), U16.7 (GND), U17.7 (GND), U18.7 (GND), U19.7 (GND), U6.21 (CLK2), U6.22 (DRV), U6.31 (GND), U7.5 (GND), U8.8 (GND), U9.8 (GND); no longer U4.36 (~CTS)
- net PC3: now also U7.20 (CLK/TRG3)
- net RESET: now also U16.11, U16.12, U6.19 (RST); no longer U16.2, U16.3
- net RTC_CLK: now also U10.15 (Q5); no longer U10.10 (Q3)
- net RTC_IN: now also U10.5 (Q1), U13.12; no longer U10.2 (Q0), U13.5
- net RTC_IO: now also U13.11, U13.9; no longer U13.2, U13.6
- net RTC_PLUP: now also U13.2; no longer U13.9
- net RTC_WE: now also U10.2 (Q0), U13.13; no longer U10.5 (Q1), U13.4
- net RX: now also P3.2
- net TX: now also P3.3
- net UART_CLK: now also U14.11 (CLK), U18.8 (OUT)
- net UART_INT: now also U7.21 (CLK/TRG2)
- net VCC: now also U11.16 (VCC), U11.16 (VCC), U14.10 (~PR), U14.13 (~CLR), U14.14 (VCC), U14.14 (VCC), U14.4 (~PR), U16.14 (VCC), U17.11 (VCC), U17.14 (VCC), U18.11 (VCC), U18.14 (VCC), U19.11 (VCC), U19.14 (VCC), U6.24 (PCVAL), U6.40 (VCC), U6.6 (TC), U7.13 (IEI), U7.24 (VCC), U8.16 (VCC), U9.16 (VCC)
- net ~BUSRQ: now also RR4.3; no longer RR4.4
- net ~CFG_CS: now also U11.13 (B)
- net ~DC: now also U16.1; no longer U13.12
- net ~DENSEL: now also U6.36 (~RWC~/~RPM~)
- net ~DIR: now also U6.28 (~DIRC)
- net ~DOR_WR: now also U12.12 (~Y3), U15.5, U6.17 (~LDOR); no longer U15.8
- net ~DSA: now also U6.30 (~DS1)
- net ~DSB: now also U6.32 (~DS2)
- net ~FDC_CS: now also U6.3 (~CS)
- net ~HALT: now also U16.3; no longer U16.11
- net ~INDEX: now also RR1.5, U6.39 (~IDX); no longer RR1.6
- net ~INT: now also U7.12 (~INT)
- net ~IORQ: now also U15.9, U7.10 (~IORQ)
- net ~M1: now also U16.9, U7.14 (~M1); no longer U16.5
- net ~MREQ: now also U11.1 (~G)
- net ~NMI: now also RR4.5; no longer RR4.3
- net ~RAM_CS: now also U11.5 (~Y1)
- net ~RD: now also U15.12, U15.4, U6.1 (~RD), U7.6 (~RD); no longer U15.13, U15.2
- net ~RDATA: now also U6.20 (~RDD)
- net ~RESET: now also U16.10, U14.1 (~CLR), U7.17 (~RESET); no longer U16.4
- net ~ROM_CS: now also U11.4 (~Y0)
- net ~RTC_CS: now also U15.13, U15.2; no longer U15.1, U15.4
- net ~RTC_RD: now also U13.4, U15.11; no longer U15.3
- net ~RTC_WR: now also U15.3; no longer U15.6
- net ~STEP: now also U6.29 (~STEP)
- net ~TRK0: now also RR1.6, U6.38 (~TR00); no longer RR1.5
- net ~WAIT: now also RR4.4; no longer RR4.5
- net ~WDATA: now also U6.27 (~WD)
- net ~WR: now also U15.1, U11.15 (~G), U6.2 (~WR); no longer U15.10, U15.5
- net at U21.2 (X1): now also X1.2; no longer X1.1
- net at U21.3 (X2): now also X1.1; no longer X1.2
- net ~RTS: now reaches U4.32 (~RTS)
- net ~RTS: now also U20.11 (T1IN)
- net at U16.8: now also U12.4 (~G2A); no longer R4.2
- net at U16.6: now also R4.2; no longer U12.4 (~G2A)
- net at C26.1, D1.1 (A), R2.2: now also R1.2, U16.13; no longer R1.1, U16.1
- net ~CCR_WR: now reaches U12.14 (~Y1)
- net ~CCR_WR: now also U6.18 (~LDCR)
- net ~CTC_CS: now reaches U12.15 (~Y0)
- net ~CTC_CS: now also U7.16 (~CE)
- net at U12.5 (~G2B): now also U15.8
- net at P2.2 (PM), SW1.2: now also R1.1; no longer R1.2
- net DSR renamed CTS
- net CTS: now also P3.8 (P8)
- net DTR renamed RTS
- net RTS: now also P3.7 (P7)
- net RAM_A15 renamed MA15
- net MA15: now also RR3.6, U8.9 (Q2)
- net RAM_A16 renamed MA16
- net MA16: now also RR3.4, U8.7 (Q3)
- net RAM_A17 renamed MA17
- net MA17: now also RR3.3, U8.6 (Q4)
- net RAM_A18 renamed MA18
- net MA18: now also RR2.3, U9.10 (Q1)
- removed net ~DIR_RD: U13.13, U15.11
- net ~DSR renamed ~CTS
- net ~CTS: now also U4.36 (~CTS); no longer U4.37 (~DSR)
- net ~DTR: no longer names the net of U4.33 (~DTR)
- net ~DTR: no longer U20.11 (T1IN)
- removed net ~FDC_REG: U12.12 (~Y3), U15.12, U15.9
- net ~MOTOR renamed ~MEA
- net ~MEA: now also U6.33 (~DS3~/~MO1~); no longer P5.16 (P16)
- net ~SIDE renamed ~HDSEL
- net ~HDSEL: now also U6.25 (~HS)
- net ~WGATE renamed ~WE
- net ~WE: now also U6.26 (~WE)
- net ~WRTPRO renamed ~WP
- net ~WP: now also U6.37 (~WP)
- new net: U16.4, U16.5
- new net: U7.22 (CLK/TRG1), U7.7 (ZC/TO0)
- new net: U14.12 (D), U14.8 (~Q)
- new net CTC_CLK: U14.9 (Q), U7.23 (CLK/TRG0)
- new net DC: U13.5, U16.2
- new net MA14: RR3.5, U2.29 (A14), U3.3 (A14), U8.10 (Q1)
- new net MA19: RR2.6, U11.2 (A), U9.9 (Q2)
- new net MA20: RR2.5, U11.3 (B), U9.7 (Q3)
- new net MA21: RR2.4, U9.6 (Q4)
- new net RAM2_CS: U11.7 (~Y3)
- new net ~DACK: U15.6, U6.5 (~DACK)
- new net ~MEB: P5.16 (P16), U6.34 (~DS4~/~MO2~)
- new net ~PAGE_EN: U14.6 (~Q), U8.11 (~GR), U9.11 (~GR)
- new net ~PAGE_WR: U11.12 (~Y0), U8.12 (~GW), U9.12 (~GW)
- new net ~PGEN_WR: U11.11 (~Y1), U14.3 (CLK)
- new net ~RAM1_CS: U11.6 (~Y2)
Other:
- note added: "(Z80 CPU)"
- note added: "(Z80 CTC)"
- note added: "MHz"
- note added: "Memory Paging"
- note added: "Pull-up and Pull-down Resistors"
- note added: "Timer"
- note removed: "Interrupts"
- note removed: "Memory Paging Logic"
- note removed: "Pull-up Resistors"
- moved on the sheet: BT1, C1, C10, C11, C12, C13, C14, C15, C16, C17, C18, C19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
